Commit message: remove panda_hand; restore moveit_controller_manager

File: src/dual_panda_description/urdf/panda.urdf.xacro (robot description, xacro)
@@ -207,79 +207,4 @@
         <axis xyz="0 0 0" />
     </joint>
-    <joint name="${prefix}panda_hand_joint" type="fixed">
-        <parent link="${prefix}panda_link8" />
-        <child link="${prefix}panda_hand" />
-        <origin rpy="0 0 -0.785398163397" xyz="0 0 0" />
-    </joint>
-    <link name="${prefix}panda_hand">
-        <visual>
-            <geometry>
-                <mesh filename="file://$(find moveit_resources_panda_description)/meshes/visual/hand.dae" />
-            </geometry>
-        </visual>
-        <collision>
-            <geometry>
-                <mesh filename="file://$(find moveit_resources_panda_description)/meshes/collision/hand.stl" />
-            </geometry>
-        </collision>
-        <inertial>
-          <origin xyz="-0.01 0 0.03" rpy="0 0 0" />
-          <mass value="0.73"/>
-          <inertia ixx="0.001" iyy="0.0025" izz="0.0017" ixy="0" ixz="0" iyz="0"/>
-        </inertial>
-    </link>
-    <link name="${prefix}panda_leftfinger">
-        <visual>
-            <geometry>
-                <mesh filename="file://$(find moveit_resources_panda_description)/meshes/visual/finger.dae" />
-            </geometry>
-        </visual>
-        <collision>
-            <geometry>
-                <mesh filename="file://$(find moveit_resources_panda_description)/meshes/collision/finger.stl" />
-            </geometry>
-        </collision>
-        <inertial>
-          <origin xyz="0 0 0" rpy="0 0 0" />
-          <mass value="0.015"/>
-          <inertia ixx="2.375E-6" iyy="2.375E-6" izz="7.5E-7" ixy="0" ixz="0" iyz="0"/>
-        </inertial>
-    </link>
-    <link name="${prefix}panda_rightfinger">
-        <visual>
-            <origin rpy="0 0 3.14159265359" xyz="0 0 0" />
-            <geometry>
-                <mesh filename="file://$(find moveit_resources_panda_description)/meshes/visual/finger.dae" />
-            </geometry>
-        </visual>
-        <collision>
-            <origin rpy="0 0 3.14159265359" xyz="0 0 0" />
-            <geometry>
-                <mesh filename="file://$(find moveit_resources_panda_description)/meshes/collision/finger.stl" />
-            </geometry>
-        </collision>
-        <inertial>
-          <origin xyz="0 0 0" rpy="0 0 0" />
-          <mass value="0.15"/>
-          <inertia ixx="2.375E-6" iyy="2.375E-6" izz="7.5E-7" ixy="0" ixz="0" iyz="0"/>
-        </inertial>
-    </link>
-    <joint name="${prefix}panda_finger_joint1" type="prismatic">
-        <parent link="${prefix}panda_hand" />
-        <child link="${prefix}panda_leftfinger" />
-        <origin rpy="0 0 0" xyz="0 0 0.0584" />
-        <axis xyz="0 1 0" />
-        <limit effort="20" lower="0.0" upper="0.04" velocity="0.2" />
-        <dynamics damping="0.3" />
-    </joint>
-    <joint name="${prefix}panda_finger_joint2" type="prismatic">
-        <parent link="${prefix}panda_hand" />
-        <child link="${prefix}panda_rightfinger" />
-        <origin rpy="0 0 0" xyz="0 0 0.0584" />
-        <axis xyz="0 -1 0" />
-        <limit effort="20" lower="0.0" upper="0.04" velocity="0.2" />
-        <mimic joint="${prefix}panda_finger_joint1" />
-        <dynamics damping="0.3" />
-    </joint>
     </xacro:macro>
 </robot>
